File: Io.brd (EAGLE design)
At the start: 99.7 x 76.2 mm, 101 parts, among them IC1 AT90CAN128, IC2 MCP2551SO8, IC3 NUP2105L, IC5 LD117ADT50TR, J1 POWER_JACKPTH, Q1 56P2859, Q2 PMV56XN, Q3 PMV56XN, Q4 PMV56XN, Q5 PMV56XN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

Commit message: Io 20120215
Parts:
- removed U$10: (no value), OpenLCB:NMRA_ORG_SMALL
- removed U$2: (no value), Iodph:ARTIFICIAL_SCIENCE_RAILSTARS_50MM_INV
- C1, C10, C11, C12, C16, C2, C4, C5, C6, C7, C8, C9: device rcl:C1206 -> rcl:C0805
- LED1, LED10, LED11, LED2, LED3, LED4, LED5, LED6, LED7, LED8, LED9: device led:CHIPLED_1206 -> led:CHIP-LED0805
- R1, R10, R11, R12, R13, R14, R15, R16, R17, R18, R19, R2, R20, R21, R22, R23, R24, R25, R26, R3, R6, R7, R8, R9: device rcl:R1206 -> rcl:R0805
- U$4: value (none) -> RAILSTARS_LOGO50MM; device Iodph:OPENLCB_NMRANET_LOGO_MED -> Artificial Science:RAILSTARS_50MM
- moved U$4 94.7 mm to (97.2, 18.4), flipped to the bottom
- moved U$7 44.6 mm to (52.9, 12.4)
- moved U$1 5.00 mm to (54.8, 26.4)
- moved U$9 5.00 mm to (1.91, 12.0)
- moved U$13 0.64 mm to (27.9, 16.2)
- turned JP9 to 270 degrees
- turned R18 to 270 degrees
- turned R19 to 270 degrees
- turned R20 to 270 degrees
- turned R21 to 270 degrees
- turned R22 to 270 degrees
- turned R23 to 270 degrees
- turned R24 to 270 degrees
- turned R25 to 270 degrees
Routing:
- net TX: track 77.0 -> 68.7 mm
- net RESET: track 57.9 -> 62.6 mm
- net PB1: track 52.1 -> 55.7 mm
- net GND: track 124.2 -> 126.7 mm
- net N$21: track 5.12 -> 3.85 mm
- net N$15: track 5.12 -> 3.85 mm
- net N$20: track 5.12 -> 3.85 mm
- net N$19: track 5.12 -> 3.85 mm
- net N$14: track 5.12 -> 3.85 mm
- net N$13: track 5.12 -> 3.85 mm
- net N$18: track 5.12 -> 3.85 mm
- net N$17: track 5.12 -> 3.85 mm
- net PG0: track 25.1 -> 26.1 mm
- net PG1: track 26.9 -> 28.0 mm
- net N$5: track 3.72 -> 4.48 mm
Other:
- board text added: "05.02.01.02.03."
- board text added: "20120215"
- board text added: "44652"
- board text added: "Copyright (C) 2012 D.E. Goodman-Wilson"
- board text added: "http://railstars.com/hardware/io/io-developers-board/"
- board text removed: "05.02.01.02.02."
- board text removed: "20120103"
- board text removed: "Copyright (C) 2011 D.E. Goodman-Wilson"
- board text removed: "NMRAnet S-9.7"
- board text removed: "http://railstars.com/hardware/io"
- board text removed: "v1.0"
