File: Io.sch (EAGLE design)
At the start: 91 parts, among them IC1 AT90CAN128, IC2 MCP2551SO8, IC3 NUP2105L, IC5 LD117ADT50TR, J1 POWER_JACKPTH, Q1 56P2859, Q2 PMV56XN, Q3 PMV56XN, Q4 PMV56XN, Q5 PMV56XN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

Commit message: Io 20120215
Parts:
- added U$4: RAILSTARS_LOGO50MM, Artificial Science:RAILSTARS_LOGO50MM
- C1, C10, C11, C12, C16, C2, C4, C5, C6, C7, C8, C9: device rcl:C-USC1206 -> rcl:C-USC0805
- LED1, LED10, LED11, LED2, LED3, LED4, LED5, LED6, LED7, LED8, LED9: device led:LEDCHIPLED_1206 -> led:LEDCHIP-LED0805
- R1, R10, R11, R12, R13, R14, R15, R16, R17, R18, R19, R2, R20, R21, R22, R23, R24, R25, R26, R3, R6, R7, R8, R9: device rcl:R-US_R1206 -> rcl:R-US_R0805
Other:
- note added: "/hardware/io/io-developers-board/"
- note added: "12"
- note added: "12 02 15"
- note added: "Io Developer's Board"
- note removed: ""Io" NMRAnet 8-Line I/O Board"
- note removed: "/hardware/io"
- note removed: "11"
- note removed: "2011 12 31"
